File: mfosish_ww_supply/mfosish_ww_supply.kicad_pcb (KiCad board)
At the start: 2 copper layers, 100 x 61 mm, 35 parts, among them J1 Conn_01x03, J2 Conn_01x02, J3 Conn_01x02, J4 Conn_01x03, U1 LM7812_TO220, U2 LM7912_TO220

Commit message: extend board outline to allpcb free limits
Parts:
- moved H1 1.00 mm to (53.0, 68.0)
- moved H2 1.00 mm to (147.0, 68.0)
- moved H4 0.05 mm to (146.9, 122.0)
Other:
- board size 100 x 61 mm -> 250 x 60 mm

Commit message: insert fps
Parts:
- added J10: Synth_power_2x5, ao_tht:Power_Header, F.Cu at (224.9, 78.0)
- added J11: Synth_power_2x5, ao_tht:Power_Header, F.Cu at (193.5, 100.0)
- added J12: Synth_power_2x5, ao_tht:Power_Header, F.Cu at (203.9, 100.0)
- added J13: Synth_power_2x5, ao_tht:Power_Header, F.Cu at (214.4, 100.0)
- added J14: Synth_power_2x5, ao_tht:Power_Header, F.Cu at (235.3, 78.0)
- added J15: Synth_power_2x5, ao_tht:Power_Header, F.Cu at (224.9, 100.0)
- added J16: Synth_power_2x5, ao_tht:Power_Header, F.Cu at (245.8, 78.0)
- added J5: Synth_power_2x5, ao_tht:Power_Header, F.Cu at (183.0, 78.0)
- added J6: Synth_power_2x5, ao_tht:Power_Header, F.Cu at (183.0, 100.0)
- added J7: Synth_power_2x5, ao_tht:Power_Header, F.Cu at (193.5, 78.0)
- added J8: Synth_power_2x5, ao_tht:Power_Header, F.Cu at (203.9, 78.0)
- added J9: Synth_power_2x5, ao_tht:Power_Header, F.Cu at (214.4, 78.0)

Commit message: done!
Parts:
- added H4: MountingHole, ao_tht:MountingHole_3.2mm_M3, F.Cu at (157.0, 68.0)
- added H4: MountingHole, ao_tht:MountingHole_3.2mm_M3, F.Cu at (296.0, 68.0)
- added H4: MountingHole, ao_tht:MountingHole_3.2mm_M3, F.Cu at (296.0, 122.0)
- added H4: MountingHole, ao_tht:MountingHole_3.2mm_M3, F.Cu at (157.0, 122.0)
- added J4: Conn_01x03, ao_tht:TerminalBlock_Degson_DG301_1x03_P5.00mm_Vertical, F.Cu at (157.0, 95.0)
- moved J16 52.1 mm to (291.0, 104.0)
- moved J14 44.1 mm to (279.3, 74.0)
- moved J15 42.9 mm to (267.5, 104.0)
- moved J10 31.2 mm to (255.8, 74.0)
- moved J13 29.9 mm to (244.1, 103.8)
- moved J11 27.2 mm to (185.5, 74.0)
- moved J7 26.3 mm to (197.2, 104.0)
- moved J9 18.4 mm to (232.4, 74.0)
- moved J12 17.2 mm to (220.6, 104.0)
- moved J5 14.1 mm to (169.5, 73.9)
- moved J6 10.1 mm to (173.7, 104.0)
- moved J8 6.43 mm to (208.9, 73.9)
Routing:
- net -12V: track 16.0 -> 310.5 mm
- net +12V: track 15.7 -> 305.8 mm
Other:
- outline, holes or cut-outs redrawn
- board text added: "Bus Board modification by Sonosus July 21 github.com/sonosus/ww_supply"
